File: metering.kicad_pcb (KiCad board)
At the start: 2 copper layers, 0 parts

Commit message: Create base PCBs for Camdenboss CNMB-2-2 DIN rail enclosure
Parts:
- added H1: MountingHole, MountingHole:MountingHole_3.2mm_M3, F.Cu at (89.5, 125.0)
- added H2: MountingHole, MountingHole:MountingHole_3.2mm_M3, F.Cu at (110.5, 75.0)
- added X1: Screw_Terminal_01x06, TerminalBlock_Phoenix:TerminalBlock_Phoenix_MKDS-1,5-6-5.08_1x06_P5.08mm_Horizontal, F.Cu at (87.3, 137.2)
- added X2: Screw_Terminal_01x06, TerminalBlock_Phoenix:TerminalBlock_Phoenix_MKDS-1,5-6-5.08_1x06_P5.08mm_Horizontal, F.Cu at (112.7, 62.8)
Other:
- board outline added: 68 x 129 mm
- board text added: "PCB C"
- board text added: "PCB D"
- board text added: "PCB E"
- board text added: "Smart Home Energy Metering Rev. ${REVISION}"
- board text added: "Wall"
- board text added: "https://github.com/zargony/smarthome-metering"

Commit message: PCB layout
Parts:
- added C1: 10u, Capacitor_Tantalum_SMD:CP_EIA-3216-18_Kemet-A, F.Cu at (74.5, 121.0)
- added C10: 100n, Capacitor_SMD:C_0805_2012Metric, F.Cu at (60.5, 74.0)
- added C11: 100n, Capacitor_SMD:C_0805_2012Metric, F.Cu at (67.5, 74.0)
- added C12: 100n, Capacitor_SMD:C_0805_2012Metric, F.Cu at (74.5, 74.0)
- added C13: 100n, Capacitor_SMD:C_0805_2012Metric, F.Cu at (57.5, 72.0)
- added C2: 22u, Capacitor_Tantalum_SMD:CP_EIA-3216-18_Kemet-A, F.Cu at (77.5, 121.0)
- added C3: TBD, Capacitor_SMD:C_0805_2012Metric, F.Cu at (54.5, 112.0)
- added C4: TBD, Capacitor_SMD:C_0805_2012Metric, F.Cu at (60.5, 112.0)
- added C5: 10u, Capacitor_Tantalum_SMD:CP_EIA-3216-18_Kemet-A, F.Cu at (63.5, 89.0)
- added C6: 100n, Capacitor_SMD:C_0805_2012Metric, F.Cu at (64.0, 86.5)
- added C7: 12p, Capacitor_SMD:C_0805_2012Metric, F.Cu at (72.0, 112.5)
- added C8: 12p, Capacitor_SMD:C_0805_2012Metric, F.Cu at (72.0, 114.5)
- added C9: 1u, Capacitor_SMD:C_0805_2012Metric, F.Cu at (62.0, 83.5)
- added D1: SS12, Diode_SMD:D_SMA, F.Cu at (75.0, 126.5)
- added D10: LED, LED_THT:LED_D3.0mm, F.Cu at (44.5, 108.7)
- added D2: SS12, Diode_SMD:D_SMA, F.Cu at (67.0, 126.5)
- added D3: LED, LED_THT:LED_D3.0mm, F.Cu at (44.5, 93.7)
- added D4: LED, LED_THT:LED_D3.0mm, F.Cu at (44.5, 88.7)
- added D5: 1N4148W, Diode_SMD:D_SOD-123, F.Cu at (61.0, 80.5)
- added D6: LED, LED_THT:LED_D3.0mm, F.Cu at (44.5, 98.7)
- added D7: 1N4148W, Diode_SMD:D_SOD-123, F.Cu at (68.0, 80.5)
- added D8: LED, LED_THT:LED_D3.0mm, F.Cu at (44.5, 103.7)
- added D9: 1N4148W, Diode_SMD:D_SOD-123, F.Cu at (75.0, 80.5)
- added J1: Conn_01x08, Connector_PinSocket_2.54mm:PinSocket_1x08_P2.54mm_Vertical, F.Cu at (90.2, 91.1)
- added J2: USB_C_Receptacle_USB2.0_16P, Connector_USB:USB_C_Receptacle_GCT_USB4110, F.Cu at (54.5, 126.1)
- added J3: Prog, Connector_PinHeader_2.54mm:PinHeader_1x04_P2.54mm_Vertical, F.Cu at (68.7, 86.5)
- added P1: Conn_01x08, Connector_PinHeader_2.54mm:PinHeader_1x08_P2.54mm_Horizontal, F.Cu at (68.6, 91.1)
- added R1: 5k1, Resistor_SMD:R_0805_2012Metric, F.Cu at (60.5, 117.5)
- added R10: 1k, Resistor_SMD:R_0805_2012Metric, F.Cu at (48.5, 95.0)
- added R11: 0, Resistor_SMD:R_0805_2012Metric, F.Cu at (58.0, 85.0)
- added R12: 10k, Resistor_SMD:R_0805_2012Metric, F.Cu at (64.0, 83.5)
- added R13: 10k, Resistor_SMD:R_0805_2012Metric, F.Cu at (46.0, 119.0)
- added R14: 1k, Resistor_SMD:R_0805_2012Metric, F.Cu at (48.5, 90.0)
- added R15: 10k, Resistor_SMD:R_0805_2012Metric, F.Cu at (60.5, 76.0)
- added R16: 10k, Resistor_SMD:R_0805_2012Metric, F.Cu at (60.5, 78.0)
- added R17: 1k, Resistor_SMD:R_0805_2012Metric, F.Cu at (48.5, 100.0)
- added R18: 10k, Resistor_SMD:R_0805_2012Metric, F.Cu at (67.5, 76.0)
- added R19: 10k, Resistor_SMD:R_0805_2012Metric, F.Cu at (67.5, 78.0)
- added R2: 5k1, Resistor_SMD:R_0805_2012Metric, F.Cu at (58.5, 117.5)
- added R20: 1k, Resistor_SMD:R_0805_2012Metric, F.Cu at (48.5, 105.0)
- added R21: 10k, Resistor_SMD:R_0805_2012Metric, F.Cu at (74.5, 76.0)
- added R22: 10k, Resistor_SMD:R_0805_2012Metric, F.Cu at (74.5, 78.0)
- added R23: 1k, Resistor_SMD:R_0805_2012Metric, F.Cu at (48.5, 110.0)
- added R3: 10k, Resistor_SMD:R_0805_2012Metric, F.Cu at (77.5, 113.0)
- added R4: 499, Resistor_SMD:R_0805_2012Metric, F.Cu at (55.5, 89.0)
- added R5: 0, Resistor_SMD:R_0805_2012Metric, F.Cu at (56.5, 112.0)
- added R6: 0, Resistor_SMD:R_0805_2012Metric, F.Cu at (58.5, 112.0)
- added R7: 0, Resistor_SMD:R_0805_2012Metric, F.Cu at (64.8, 112.0)
- added R8: 0, Resistor_SMD:R_0805_2012Metric, F.Cu at (62.8, 112.0)
- added R9: NC, Resistor_SMD:R_0805_2012Metric, F.Cu at (66.8, 113.4)
- added SW1: Reset, Button_Switch_SMD:SW_Tactile_SPST_NO_Straight_CK_PTS636Sx25SMTRLFS, F.Cu at (47.5, 84.5)
- added SW2: Boot, Button_Switch_SMD:SW_Tactile_SPST_NO_Straight_CK_PTS636Sx25SMTRLFS, F.Cu at (47.5, 115.5)
- added U1: USBLC6-2SC6, Package_TO_SOT_SMD:SOT-23-6, F.Cu at (54.5, 117.5)
- added U2: AMS1117-3.3, Package_TO_SOT_SMD:SOT-223-3_TabPin2, F.Cu at (68.0, 121.0)
- added U3: ESP32-C3-WROOM-02U, RF_Module:ESP32-C3-WROOM-02U, F.Cu at (58.2, 100.0)
- added U4: 74HC14, Package_SO:SOIC-14_3.9x8.7mm_P1.27mm, F.Cu at (53.0, 77.5)
- added Y1: 32.768kHz, Crystal:Crystal_SMD_3215-2Pin_3.2x1.5mm, F.Cu at (69.0, 113.5)
Connections:
- net GND renamed GND1
- X1 pad 4: +3.3V -> Net-(J1-Pin_3)
- X1 pad 5: /UART_RX -> Net-(J1-Pin_4)
- X1 pad 6: /UART_TX -> Net-(J1-Pin_5)
- X2 pad 2: /CONTACT1 -> Net-(J1-Pin_6)
- X2 pad 4: /CONTACT2 -> Net-(J1-Pin_7)
- X2 pad 6: /CONTACT3 -> Net-(J1-Pin_8)
Routing:
- net +3.3V: track 0.00 -> 190.4 mm, vias 0 -> 6
- net Net-(J1-Pin_5): track 0.00 -> 61.3 mm
- net Net-(J1-Pin_4): track 0.00 -> 60.5 mm
- net Net-(J1-Pin_3): track 0.00 -> 60.0 mm
- net Net-(J1-Pin_8): track 0.00 -> 58.4 mm, vias 0 -> 1
- net Net-(J1-Pin_6): track 0.00 -> 57.6 mm, vias 0 -> 1
- net /CONTACT1: track 0.00 -> 54.8 mm
- net /IO4: track 0.00 -> 54.3 mm, vias 0 -> 2
- net /IO5: track 0.00 -> 51.8 mm, vias 0 -> 2
- net /CONTACT2: track 0.00 -> 51.6 mm
- net Net-(J1-Pin_7): track 0.00 -> 50.0 mm, vias 0 -> 1
- net Net-(J1-Pin_2): track 0.00 -> 48.8 mm
- net /CONTACT3: track 0.00 -> 48.1 mm
- net /VIN: track 0.00 -> 46.4 mm, vias 0 -> 1
- net /IO3: track 0.00 -> 46.3 mm, vias 0 -> 4
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- added copper zone on B.Cu, net GND
- added copper zone on F.Cu, net GND
- added copper zone on B.Cu, net GND1
- added copper zone on F.Cu, net GND1
Other:
- board size 68 x 129 mm -> 75 x 86 mm
- board text added: "+ 5V IN -"
- board text added: "3.3V"
- board text added: "5V"
- board text added: "Cnt1"
- board text added: "Cnt2"
- board text added: "Cnt3"
- board text added: "Energy Metering Rev. ${REVISION}"
- board text added: "GND"
- board text added: "Rx"
- board text added: "Tx"
- board text added: "github.com/zargony/smarthome-metering"
- board text removed: "PCB C"
- board text removed: "Smart Home Energy Metering Rev. ${REVISION}"
- board text removed: "https://github.com/zargony/smarthome-metering"
