File: debounce.kicad_sch (KiCad schematic)
At the start: 7 parts, among them U4 74HC14

Commit message: Clear PCB and prepare layout for CNMB-3-2
Other:
- title: Smart Home Energy Metering -> Smart Home Metering
Changed lines of the file:
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@@
 	(paper "A4")
 	(title_block
-		(title "Smart Home Energy Metering")
-		(date "2025-08-01")
+		(title "Smart Home Metering")
+		(date "2026-09-20")
 		(rev "1.2")
 		(comment 1 "https://github.com/zargony/smarthome-metering")
